Commit message: feat: add asg_03 package

File: ros_101_gazebo_rviz/urdf/robot_tutorial.xacro (robot description, xacro)
@@ -125,4 +125,27 @@
     <origin xyz="${caster_wheel_joint_offset} 0 -${caster_wheel_radius+0.005}" rpy="0 0 0"/>
   </joint>
+  <!--Laser Joint-->
+  <joint name="laser_joint" type="fixed">
+    <axis xyz="0 1 0"/>
+    <origin xyz="0.075 0 0.02" rpy="0 0 0"/>
+    <parent link="base_link"/>
+    <child link="laser_link"/>
+  </joint>
+  <!--Laser Link-->
+  <link name="laser_link">
+    <collision>
+      <origin xyz="0 0 0" rpy="0 0 0"/>
+      <geometry>
+        <box size="0.025 0.025 0.025"/>
+      </geometry>
+    </collision>
+    <visual>
+      <origin xyz="0 0 0" rpy="0 0 0"/>
+      <geometry>
+        <box size="0.025 0.025 0.025"/>
+      </geometry>
+    </visual>
+    <xacro:box_inertia m="1" w="0.025" h="0.025" d="0.025"/>
+  </link>
   <xacro:include filename="$(find ros_101_gazebo_rviz)/urdf/robot_tutorial_gazebo.xacro"/>
 </robot>

File: ros_101_gazebo_rviz/urdf/robot_tutorial_gazebo.xacro (robot description, xacro)
@@ -17,4 +17,34 @@
     </plugin>
   </gazebo>
+   <gazebo reference="laser_link">
+    <sensor type="ray" name="laser_sensor">
+      <pose>0 0 0 0 0 0</pose>
+      <visualize>true</visualize>
+      <update_rate>40</update_rate>
+      <ray>
+        <scan>
+          <horizontal>
+            <samples>5</samples>
+            <min_angle>-0.0349066</min_angle>
+            <max_angle>0.0349066</max_angle>
+          </horizontal>
+        </scan>
+        <range>
+          <min>0.10</min>
+          <max>30.0</max>
+          <resolution>0.01</resolution>
+        </range>
+        <noise>
+          <type>gaussian</type>
+          <mean>0.0</mean>
+          <stddev>0.01</stddev>
+        </noise>
+      </ray>
+      <plugin name="gazebo_ros_head_hokuyo_controller" filename="libgazebo_ros_laser.so">
+        <topicName>/scan</topicName>
+        <frameName>laser_link</frameName>
+      </plugin>
+    </sensor>
+  </gazebo>
   <gazebo reference="base_link">
     <material>Gazebo/White</material>
