Commit message: feat: add left and right scanner

File: asg_04/urdf/robot_tutorial.xacro (robot description, xacro)
@@ -148,4 +148,50 @@
     <xacro:box_inertia m="1" w="0.025" h="0.025" d="0.025"/>
   </link>
-  <xacro:include filename="$(find ros_101_gazebo_rviz)/urdf/robot_tutorial_gazebo.xacro"/>
+    <!--Left Laser Joint-->
+  <joint name="left_laser_joint" type="fixed">
+    <axis xyz="0 1 0"/>
+    <origin xyz="0.075 0.05 0.02" rpy="0 0 0.52"/>
+    <parent link="base_link"/>
+    <child link="left_laser_link"/>
+  </joint>
+  <!--Left Laser Link-->
+  <link name="left_laser_link">
+    <collision>
+      <origin xyz="0 0 0" rpy="0 0 0"/>
+      <geometry>
+        <box size="0.025 0.025 0.025"/>
+      </geometry>
+    </collision>
+    <visual>
+      <origin xyz="0 0 0" rpy="0 0 0"/>
+      <geometry>
+        <box size="0.025 0.025 0.025"/>
+      </geometry>
+    </visual>
+    <xacro:box_inertia m="1" w="0.025" h="0.025" d="0.025"/>
+  </link>
+  <!--Right Laser Joint-->
+  <joint name="right_laser_joint" type="fixed">
+    <axis xyz="0 1 0"/>
+    <origin xyz="0.075 -0.05 0.02" rpy="0 0 -0.52"/>
+    <parent link="base_link"/>
+    <child link="right_laser_link"/>
+  </joint>
+  <!--Right Laser Link-->
+  <link name="right_laser_link">
+    <collision>
+      <origin xyz="0 0 0" rpy="0 0 0"/>
+      <geometry>
+        <box size="0.025 0.025 0.025"/>
+      </geometry>
+    </collision>
+    <visual>
+      <origin xyz="0 0 0" rpy="0 0 0"/>
+      <geometry>
+        <box size="0.025 0.025 0.025"/>
+      </geometry>
+    </visual>
+    <xacro:box_inertia m="1" w="0.025" h="0.025" d="0.025"/>
+  </link>
+  <xacro:include filename="$(find asg_04)/urdf/robot_tutorial_gazebo.xacro"/>
 </robot>

File: asg_04/urdf/robot_tutorial_gazebo.xacro (robot description, xacro)
@@ -42,6 +42,66 @@
       </ray>
       <plugin name="gazebo_ros_head_hokuyo_controller" filename="libgazebo_ros_laser.so">
-        <topicName>/scan</topicName>
-        <frameName>laser_link</frameName>
+        <topicName>/scan_center</topicName>
+        <frameName>center_laser_link</frameName>
+      </plugin>
+    </sensor>
+  </gazebo>
+  <gazebo reference="left_laser_link">
+    <sensor type="ray" name="laser_sensor">
+      <pose>0 0 0 0 0 0</pose>
+      <visualize>true</visualize>
+      <update_rate>40</update_rate>
+      <ray>
+        <scan>
+          <horizontal>
+            <samples>5</samples>
+            <min_angle>-0.0349066</min_angle>
+            <max_angle>0.0349066</max_angle>
+          </horizontal>
+        </scan>
+        <range>
+          <min>0.10</min>
+          <max>30.0</max>
+          <resolution>0.01</resolution>
+        </range>
+        <noise>
+          <type>gaussian</type>
+          <mean>0.0</mean>
+          <stddev>0.01</stddev>
+        </noise>
+      </ray>
+      <plugin name="gazebo_ros_head_hokuyo_controller" filename="libgazebo_ros_laser.so">
+        <topicName>/scan_left</topicName>
+        <frameName>left_laser_link</frameName>
+      </plugin>
+    </sensor>
+  </gazebo>
+  <gazebo reference="right_laser_link">
+    <sensor type="ray" name="laser_sensor">
+      <pose>0 0 0 0 0 0</pose>
+      <visualize>true</visualize>
+      <update_rate>40</update_rate>
+      <ray>
+        <scan>
+          <horizontal>
+            <samples>5</samples>
+            <min_angle>-0.0349066</min_angle>
+            <max_angle>0.0349066</max_angle>
+          </horizontal>
+        </scan>
+        <range>
+          <min>0.10</min>
+          <max>30.0</max>
+          <resolution>0.01</resolution>
+        </range>
+        <noise>
+          <type>gaussian</type>
+          <mean>0.0</mean>
+          <stddev>0.01</stddev>
+        </noise>
+      </ray>
+      <plugin name="gazebo_ros_head_hokuyo_controller" filename="libgazebo_ros_laser.so">
+        <topicName>/scan_right</topicName>
+        <frameName>right_laser_link</frameName>
       </plugin>
     </sensor>

File: asg_04/urdf/test.urdf (robot description, URDF)
Before this commit: robot robot_tutorial, 6 links, 5 joints
Links:
- added link left_laser_link, mass 1; collision box size=0.025 0.025 0.025; visual box size=0.025 0.025 0.025
- added link right_laser_link, mass 1; collision box size=0.025 0.025 0.025; visual box size=0.025 0.025 0.025
Joints:
- added joint left_laser_joint: type fixed, parent base_link, child right_laser_link, origin xyz=0.075 -0.05 0.02 rpy=0 0 330, axis 0 1 0
